Commit message: Added URDF stuff

File: Simulation/PyBullet/urdf_files/dodo_simple.urdf (robot description, URDF)
Before this commit: robot Dodo, 4 links, 3 joints
Links:
- link toe: geometry collision sphere radius=0.1; visual sphere radius=0.1

File: Simulation/PyBullet/urdf_files/dodo_simple_vertical_test_stand.urdf (robot description, URDF)
Before this commit: robot Dodo, 4 links, 3 joints
Links:
- added link toe, mass 5; collision sphere radius=0.1; visual sphere radius=0.1
- link base_link: mass None -> 1
Joints:
- added joint link_2_to_toe: type fixed, parent link_2, child toe, origin xyz=0 0 -1.0
- joint base_link_to_body: limit lower=-10 upper=10 effort=10 velocity=10 -> effort=100000 velocity=100000
- joint body_to_link_1: limit effort=10 velocity=10 -> effort=100000 velocity=100000
- joint link_1_to_link_2: limit effort=10 velocity=10 -> effort=100000 velocity=100000

Commit message: Worked on vertical test bed / test case 2, will continue later to implement proper motor control to prevent the body from pitching forward or backwards.

File: Simulation/PyBullet/urdf_files/dodo_simple.urdf (robot description, URDF)
Before this commit: robot Dodo, 4 links, 3 joints
Joints:
- joint link_2_to_toe: axis (none) -> 1 0 0; limit (none) -> effort=10 velocity=10; type fixed -> revolute
